File: src/Rotisserie-Chicken/Rotisserie-Chicken.kicad_sch (KiCad schematic)
At the start: 9 parts, among them P1 282837-6, P2 647676-2

Commit message: routed PCB
Parts:
- D1: footprint (none) -> Rotisserie-Chicken:LED
Changed lines of the file:
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@@
       (effects (font (size 1.524 1.524)) (justify left))
     )
-    (property "Footprint" "" (id 2) (at 190.5 91.059 0)
+    (property "Footprint" "Rotisserie-Chicken:LED" (id 2) (at 190.5 91.059 0)
       (effects (font (size 1.524 1.524)) hide)
     )
@@
     )
     (path "/836be2cc-0648-4199-97ea-3b453b6d3878"
-      (reference "D1") (unit 1) (value "LED") (footprint "")
+      (reference "D1") (unit 1) (value "LED") (footprint "Rotisserie-Chicken:LED")
     )
     (path "/3f55e6d7-7f6d-4e6b-af8a-5d85d2fe0aa1"
