File: src/Rotisserie-Chicken/Rotisserie-Chicken.kicad_pcb (KiCad board)
At the start: 2 copper layers, 50.5 x 38.6 mm, 9 parts, among them P1 282837-6, P2 647676-2

Commit message: added labels to screw terminals
Other:
- board text added: "+"
- board text added: "-"
- board text added: "Arduino"
- board text added: "Motor"
- board text added: "Power"
Changed lines of the file:
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@@
   (gr_line (start 76.454 102.108) (end 76.454 63.5) (layer "Edge.Cuts") (width 0.1))
   (gr_line (start 127 102.108) (end 76.454 102.108) (layer "Edge.Cuts") (width 0.1))
+  (gr_text "+\n\n\n" (at 114.935 100.33) (layer "F.SilkS")
+    (effects (font (size 1 1) (thickness 0.15)))
+  )
+  (gr_text "Power" (at 102.108 100.711) (layer "F.SilkS")
+    (effects (font (size 1 1) (thickness 0.15)))
+  )
+  (gr_text "Arduino\n" (at 112.649 100.711) (layer "F.SilkS")
+    (effects (font (size 1 1) (thickness 0.15)))
+  )
+  (gr_text "Motor\n" (at 91.44 100.584) (layer "F.SilkS")
+    (effects (font (size 1 1) (thickness 0.15)))
+  )
+  (gr_text "-\n\n" (at 99.441 99.187) (layer "F.SilkS")
+    (effects (font (size 1 1) (thickness 0.15)))
+  )
+  (gr_text "+\n\n\n" (at 104.648 100.076) (layer "F.SilkS")
+    (effects (font (size 1 1) (thickness 0.15)))
+  )
+  (gr_text "-\n\n" (at 110.109 99.568) (layer "F.SilkS")
+    (effects (font (size 1 1) (thickness 0.15)))
+  )
+  (gr_text "+\n\n\n" (at 94.488 100.076) (layer "F.SilkS")
+    (effects (font (size 1 1) (thickness 0.15)))
+  )
+  (gr_text "-\n\n" (at 89.281 99.187) (layer "F.SilkS")
+    (effects (font (size 1 1) (thickness 0.15)))
+  )
   (segment (start 118.618 74.549) (end 118.618 91.948) (width 0.508) (layer "F.Cu") (net 1))
   (segment (start 100.411 69.596) (end 113.665 69.596) (width 0.508) (layer "F.Cu") (net 1))
